Commit message: Modified dlr vessel description

File: dlr_sensors/urdf/GNSS_MTi_680G.urdf.xacro (robot description, xacro)
@@ -44,5 +44,5 @@
             </inertial> -->
         </link>
-        <gazebo>
+        <!-- <gazebo>
             <plugin name="${prefix}_imu_plugin" filename="libgazebo_ros_imu.so">
                 <alwaysOn>true</alwaysOn>
@@ -51,6 +51,26 @@
                 <serviceName>imu_service</serviceName>
                 <gaussianNoise>0.004</gaussianNoise>
-                <updateRate>20.0</updateRate>
+                <updateRate>50.0</updateRate>
             </plugin>
+        </gazebo> -->
+        <gazebo reference="${prefix}_base_link">
+            <gravity>true</gravity>
+            <sensor name="${prefix}_imu_sensor" type="imu">
+                <always_on>true</always_on>
+                <update_rate>100</update_rate>
+                <visualize>true</visualize>
+                <topic>__default_topic__</topic>
+                <plugin filename="libgazebo_ros_imu_sensor.so" name="${prefix}_imu_plugin">
+                    <topicName>imu/data</topicName>
+                    <bodyName>${prefix}_base_link</bodyName>
+                    <updateRateHZ>100.0</updateRateHZ>
+                    <gaussianNoise>0.0</gaussianNoise>
+                    <xyzOffset>0 0 0</xyzOffset>
+                    <rpyOffset>0 0 0</rpyOffset>
+                    <frameName>${prefix}_base_link</frameName>
+                    <initialOrientationAsReference>false</initialOrientationAsReference>
+                </plugin>
+                <pose>0 0 0 0 0 0</pose>
+            </sensor>
         </gazebo>
     </xacro:macro>

File: dlr_vessel_description/robots/dlr_vessel.xacro (robot description, xacro)
@@ -13,5 +13,5 @@
         collision_range="0.3" min_range="0.9" max_range="130.0"
         noise="0.008" min_angle="-${M_PI}" max_angle="${M_PI}" gpu="false">
-        <origin xyz="9.75 0 2.15" rpy="0 0 0"/>
+        <origin xyz="9.75 0 2.20" rpy="0 0 0"/>
     </xacro:VLP-16>
     <!-- Include Stereolab Zed2 camera -->
@@ -20,5 +20,5 @@
     <xacro:include filename="$(find dlr_sensors)/urdf/stereolabs_zed2.urdf.xacro" />
     <xacro:stereolabs_zed2 camera_name_prefix="$(arg camera_name)" parent="$(arg model_name)_base_link" enable_gazebo_plugin="$(arg enable_gazebo_plugin)">
-        <origin xyz="9.75 0 2.25" rpy="0 0 0"/>
+        <origin xyz="9.75 0 2.35" rpy="0 0 0"/>
     </xacro:stereolabs_zed2>
     <!-- Include GNSS MTi 680G imu -->
@@ -27,5 +27,5 @@
     <xacro:include filename="$(find dlr_sensors)/urdf/GNSS_MTi_680G.urdf.xacro" />
     <xacro:gnss_mti_680g prefix="$(arg imu_name)" parent="$(arg model_name)_base_link">
-        <origin xyz="9.75 0 4.25" rpy="0 0 0"/>
+        <origin xyz="9.75 0 2.4" rpy="0 0 0"/>
     </xacro:gnss_mti_680g>
 </robot>

File: dlr_vessel_description/urdf/dlr_vessel.urdf.xacro (robot description, xacro)
@@ -31,5 +31,5 @@
             </visual>
             <collision>
-                <origin xyz="0 0 0.05" rpy="0 0 0"/>
+                <origin xyz="0 0 0" rpy="0 0 0"/>
                 <geometry>
                     <mesh filename="package://dlr_vessel_description/meshes/patrol_boat.stl"/>
@@ -43,14 +43,14 @@
         <!-- Gazebo properties -->
         <gazebo reference="${model_prefix}base_link">
-            <material>Gazebo/Red</material>
+            <material>Gazebo/Grey</material>
             <mu1>0.2</mu1>
             <mu2>0.2</mu2>
             <minDepth>0.001</minDepth>
             <maxVel>0</maxVel>
-            <static>true</static>
+            <!-- <static>true</static>   -->
         </gazebo>
         <!-- Adde the planar move plugin -->
         <gazebo>
-            <plugin name="object_controller" filename="libgazebo_ros_planar_move.so">
+            <plugin name="${model_prefix}planar_move_controller" filename="libgazebo_ros_planar_move.so">
             <commandTopic>cmd_vel</commandTopic>
             <odometryTopic>odom</odometryTopic>

Commit message: Added gps plugin

File: dlr_sensors/urdf/GNSS_MTi_680G.urdf.xacro (robot description, xacro)
@@ -19,7 +19,7 @@
             <xacro:insert_block name="origin" />
             <parent link="${parent}"/>
-            <child link="${prefix}_base_link" />
+            <child link="${prefix}base_link" />
         </joint>
-        <link name="${prefix}_base_link">
+        <link name="${prefix}base_link">
             <visual>
                 <origin xyz="0 0 0" rpy="0 0 0"/>
@@ -47,5 +47,5 @@
             <plugin name="${prefix}_imu_plugin" filename="libgazebo_ros_imu.so">
                 <alwaysOn>true</alwaysOn>
-                <bodyName>${prefix}_base_link</bodyName>
+                <bodyName>${prefix}base_link</bodyName>
                 <topicName>imu</topicName>
                 <serviceName>imu_service</serviceName>
@@ -54,5 +54,5 @@
             </plugin>
         </gazebo> -->
-        <gazebo reference="${prefix}_base_link">
+        <gazebo reference="${prefix}base_link">
             <gravity>true</gravity>
             <sensor name="${prefix}_imu_sensor" type="imu">
@@ -63,10 +63,10 @@
                 <plugin filename="libgazebo_ros_imu_sensor.so" name="${prefix}_imu_plugin">
                     <topicName>imu/data</topicName>
-                    <bodyName>${prefix}_base_link</bodyName>
+                    <bodyName>${prefix}base_link</bodyName>
                     <updateRateHZ>100.0</updateRateHZ>
                     <gaussianNoise>0.0</gaussianNoise>
                     <xyzOffset>0 0 0</xyzOffset>
                     <rpyOffset>0 0 0</rpyOffset>
-                    <frameName>${prefix}_base_link</frameName>
+                    <frameName>${prefix}base_link</frameName>
                     <initialOrientationAsReference>false</initialOrientationAsReference>
                 </plugin>
@@ -74,4 +74,28 @@
             </sensor>
         </gazebo>
+        <gazebo>
+            <plugin name="${prefix}_gps_plugin" filename="libhector_gazebo_ros_gps.so">
+                <updateRate>1</updateRate>
+                <!-- <robotNamespace></robotNamespace> -->
+                <bodyName>${prefix}base_link</bodyName>
+                <frameId>${prefix}base_link</frameId>
+                <topicName>gps/fix</topicName>
+                <velocityTopicName>gps/fix_velocity</velocityTopicName>
+                <referenceLatitude>49.9</referenceLatitude>
+                <referenceLongitude>8.9</referenceLongitude>
+                <referenceHeading>0.0</referenceHeading>
+                <referenceAltitude>0.0</referenceAltitude>
+                <status>0</status>
+                <service>1</service>
+                <offset>0 0 0</offset>
+                <drift>0 0 0</drift>
+                <driftFrequency>0 0 0</driftFrequency>
+                <gaussianNoise>0 0 0</gaussianNoise>
+                <velocityOffset>0 0 0</velocityOffset>
+                <velocityDrift>0 0 0</velocityDrift>
+                <velocityDriftFrequency>0 0 0</velocityDriftFrequency>
+                <velocityGaussianNoise>0 0 0</velocityGaussianNoise>
+            </plugin>
+        </gazebo>
     </xacro:macro>
 </robot>

File: dlr_vessel_description/urdf/dlr_vessel.urdf.xacro (robot description, xacro)
@@ -53,10 +53,10 @@
         <gazebo>
             <plugin name="${model_prefix}planar_move_controller" filename="libdlr_gazebo_ros_planar_move.so">
-            <commandTopic>cmd_vel</commandTopic>
-            <odometryTopic>odom</odometryTopic>
-            <odometryFrame>odom</odometryFrame>
-            <odometryRate>20.0</odometryRate>
-            <robotBaseFrame>${model_prefix}base_footprint</robotBaseFrame>
-            <robotBaseFrame>${model_prefix}base_footprint</robotBaseFrame>
+                <commandTopic>cmd_vel</commandTopic>
+                <odometryTopic>odom</odometryTopic>
+                <odometryFrame>odom</odometryFrame>
+                <odometryRate>20.0</odometryRate>
+                <robotBaseFrame>${model_prefix}base_footprint</robotBaseFrame>
+                <cmdTimeout>-1</cmdTimeout>
             </plugin>
         </gazebo>
