Commit message: Fixed dlr vessel description namespace issue

File: dlr_sensors/urdf/stereolabs_zed2.urdf.xacro (robot description, xacro)
@@ -1,5 +1,6 @@
 <?xml version="1.0"?>
 <robot name="stereolabs_zed2" xmlns:xacro="http://wiki.ros.org/xacro">
-    <xacro:macro name="stereolabs_zed2" params="camera_name_prefix:=zed
+    <xacro:macro name="stereolabs_zed2" params="prefix:=''
+                                                camera_name:=zed
                                                 parent
                                                 *origin
@@ -15,5 +16,6 @@
                 izz="${(m*(w*w+h*h))/12}"/>
     </xacro:macro>
-    <xacro:macro name="stereolabs_zed2_gazebo" params="camera_name_prefix
+    <xacro:macro name="stereolabs_zed2_gazebo" params="prefix
+                                                       camera_name
                                                        fps
                                                        baseline
@@ -24,5 +26,5 @@
                                                        near
                                                        far">
-        <gazebo reference="${camera_name_prefix}_base_link">
+        <gazebo reference="${prefix}_${camera_name}_base_link">
             <visual>
                 <material>
@@ -33,6 +35,6 @@
                 </material>
             </visual>
-            <sensor name="${camera_name_prefix}color" type="camera">
-                <camera name="${camera_name_prefix}">
+            <sensor name="${prefix}_${camera_name}color" type="camera">
+                <camera name="${prefix}_${camera_name}">
                 <horizontal_fov>${hfov}</horizontal_fov>
                 <image>
@@ -74,5 +76,5 @@
                     </noise>
                 </camera>
-                <plugin name="${camera_name_prefix}_plugin" filename="libgazebo_ros_openni_kinect.so">
+                <plugin name="${prefix}_${camera_name}_plugin" filename="libgazebo_ros_openni_kinect.so">
                     <baseline>${baseline}</baseline>
                     <alwaysOn>true</alwaysOn>
@@ -80,11 +82,11 @@
                         will control the frame rate. -->
                     <updateRate>0.0</updateRate>
-                    <cameraName>${camera_name_prefix}</cameraName>
-                    <imageTopicName>/${camera_name_prefix}/color/image_raw</imageTopicName>
-                    <cameraInfoTopicName>/${camera_name_prefix}/color/camera_info</cameraInfoTopicName>
-                    <depthImageTopicName>/${camera_name_prefix}/depth/image_raw</depthImageTopicName>
-                    <depthImageCameraInfoTopicName>/${camera_name_prefix}/depth/camera_info</depthImageCameraInfoTopicName>
-                    <pointCloudTopicName>/${camera_name_prefix}/depth/points</pointCloudTopicName>
-                    <frameName>/${camera_name_prefix}_depth_optical_frame</frameName>
+                    <cameraName>${prefix}_${camera_name}</cameraName>
+                    <imageTopicName>/${prefix}/${camera_name}/color/image_raw</imageTopicName>
+                    <cameraInfoTopicName>/${prefix}/${camera_name}/color/camera_info</cameraInfoTopicName>
+                    <depthImageTopicName>/${prefix}/${camera_name}/depth/image_raw</depthImageTopicName>
+                    <depthImageCameraInfoTopicName>/${prefix}/${camera_name}/depth/camera_info</depthImageCameraInfoTopicName>
+                    <pointCloudTopicName>/${prefix}/${camera_name}/depth/points</pointCloudTopicName>
+                    <frameName>/${prefix}_${camera_name}_depth_optical_frame</frameName>
                     <pointCloudCutoff>${near}</pointCloudCutoff>
                     <pointCloudCutoffMax>${far}</pointCloudCutoffMax>
@@ -104,10 +106,10 @@
     </xacro:macro>
         <xacro:property name="baseline" value="0.12" />
-        <joint name="${camera_name_prefix}_base_joint" type="fixed">
+        <joint name="${prefix}_${camera_name}_base_joint" type="fixed">
             <xacro:insert_block name="origin" />
             <parent link="${parent}"/>
-            <child link="${camera_name_prefix}_base_link" />
+            <child link="${prefix}_${camera_name}_base_link" />
         </joint>
-        <link name="${camera_name_prefix}_base_link">
+        <link name="${prefix}_${camera_name}_base_link">
         <visual>
             <origin xyz="0 0 0" rpy="0 0 0"/>
@@ -132,45 +134,46 @@
         </link>
         <!-- Left camera -->
-        <joint name="${camera_name_prefix}_camera_left_joint" type="fixed">
+        <joint name="${prefix}_${camera_name}_camera_left_joint" type="fixed">
             <origin xyz="0.0 0.06 0.0" rpy="0.0 0.0 0.0" />
-            <parent link="${camera_name_prefix}_base_link" />
-            <child link="${camera_name_prefix}_left_camera_frame" />
+            <parent link="${prefix}_${camera_name}_base_link" />
+            <child link="${prefix}_${camera_name}_left_camera_frame" />
         </joint>
-        <link name="${camera_name_prefix}_left_camera_frame"/>
-        <joint name="${camera_name_prefix}_camera_left_optical_joint" type="fixed">
+        <link name="${prefix}_${camera_name}_left_camera_frame"/>
+        <joint name="${prefix}_${camera_name}_camera_left_optical_joint" type="fixed">
             <origin xyz="0.0 0.0 0.0" rpy="${-M_PI/2} 0.0 ${-M_PI/2}" />
-            <parent link="${camera_name_prefix}_left_camera_frame" />
-            <child link="${camera_name_prefix}_left_camera_optical_frame" />
+            <parent link="${prefix}_${camera_name}_left_camera_frame" />
+            <child link="${prefix}_${camera_name}_left_camera_optical_frame" />
         </joint>
-        <link name="${camera_name_prefix}_left_camera_optical_frame"/>
+        <link name="${prefix}_${camera_name}_left_camera_optical_frame"/>
         <!-- Right camera-->
-        <joint name="${camera_name_prefix}_camera_right_joint" type="fixed">
+        <joint name="${prefix}_${camera_name}_camera_right_joint" type="fixed">
             <origin xyz="0.0 -0.06 0.0" rpy="0.0 0.0 0.0" />
-            <parent link="${camera_name_prefix}_base_link" />
-            <child link="${camera_name_prefix}_right_camera_frame" />
+            <parent link="${prefix}_${camera_name}_base_link" />
+            <child link="${prefix}_${camera_name}_right_camera_frame" />
         </joint>
-        <link name="${camera_name_prefix}_right_camera_frame"/>
-        <joint name="${camera_name_prefix}_camera_right_optical_joint" type="fixed">
+        <link name="${prefix}_${camera_name}_right_camera_frame"/>
+        <joint name="${prefix}_${camera_name}_camera_right_optical_joint" type="fixed">
             <origin xyz="0.0 0 0.0" rpy="${-M_PI/2} 0.0 ${-M_PI/2}" />
-            <parent link="${camera_name_prefix}_right_camera_frame" />
-            <child link="${camera_name_prefix}_right_camera_optical_frame" />
+            <parent link="${prefix}_${camera_name}_right_camera_frame" />
+            <child link="${prefix}_${camera_name}_right_camera_optical_frame" />
         </joint>
-        <link name="${camera_name_prefix}_right_camera_optical_frame"/>
+        <link name="${prefix}_${camera_name}_right_camera_optical_frame"/>
         <!-- Depth image-->
-        <joint name="${camera_name_prefix}_depth_joint" type="fixed">
+        <joint name="${prefix}_${camera_name}_depth_joint" type="fixed">
             <origin xyz="0.0 0.0 0.0" rpy="0.0 0.0 0.0" />
-            <parent link="${camera_name_prefix}_base_link" />
-            <child link="${camera_name_prefix}_depth_frame" />
+            <parent link="${prefix}_${camera_name}_base_link" />
+            <child link="${prefix}_${camera_name}_depth_frame" />
         </joint>
-        <link name="${camera_name_prefix}_depth_frame"/>
-        <joint name="${camera_name_prefix}_depth_optical_joint" type="fixed">
+        <link name="${prefix}_${camera_name}_depth_frame"/>
+        <joint name="${prefix}_${camera_name}_depth_optical_joint" type="fixed">
             <origin xyz="0.0 0.0 0.0" rpy="${-M_PI/2} 0.0 ${-M_PI/2}" />
-            <parent link="${camera_name_prefix}_depth_frame" />
-            <child link="${camera_name_prefix}_depth_optical_frame" />
+            <parent link="${prefix}_${camera_name}_depth_frame" />
+            <child link="${prefix}_${camera_name}_depth_optical_frame" />
         </joint>
-        <link name="${camera_name_prefix}_depth_optical_frame"/>
+        <link name="${prefix}_${camera_name}_depth_optical_frame"/>
         <xacro:if value="${enable_gazebo_plugin}">
             <xacro:stereolabs_zed2_gazebo
-                camera_name_prefix="${camera_name_prefix}"
+                prefix="${prefix}"
+                camera_name="${camera_name}"
                 hfov="1.2217"
                 baseline="${baseline}"

File: dlr_sensors/urdf/stereolabs_zed2_standalone.xacro (robot description, xacro)
@@ -12,5 +12,5 @@
     <link name="$(arg world_frame)"/>
     <!-- Camera macro -->
-    <xacro:stereolabs_zed2 camera_name_prefix="$(arg camera_name)" parent="$(arg world_frame)" enable_gazebo_plugin="$(arg enable_gazebo_plugin)">
+    <xacro:stereolabs_zed2 camera_name="$(arg camera_name)" parent="$(arg world_frame)" enable_gazebo_plugin="$(arg enable_gazebo_plugin)">
         <origin xyz="$(arg xyz)" rpy="$(arg rpy)"/>
     </xacro:stereolabs_zed2>

File: dlr_vessel_description/robots/dlr_vessel.xacro (robot description, xacro)
@@ -16,8 +16,8 @@
     </xacro:VLP-16>
     <!-- Include Stereolab Zed2 camera -->
-    <xacro:arg name="camera_name" default="$(arg model_name)_stereolab_zed2_camera0" />
+    <xacro:arg name="camera_name" default="stereolab_zed2_camera0" />
     <xacro:arg name="enable_gazebo_plugin" default="true" />
     <xacro:include filename="$(find dlr_sensors)/urdf/stereolabs_zed2.urdf.xacro" />
-    <xacro:stereolabs_zed2 camera_name_prefix="$(arg camera_name)" parent="$(arg model_name)_base_link" enable_gazebo_plugin="$(arg enable_gazebo_plugin)">
+    <xacro:stereolabs_zed2 prefix="$(arg model_name)" camera_name="$(arg camera_name)" parent="$(arg model_name)_base_link" enable_gazebo_plugin="$(arg enable_gazebo_plugin)">
         <origin xyz="9.75 0 2.35" rpy="0 0 0"/>
     </xacro:stereolabs_zed2>
