Commit message: Added vessel mesh

File: dlr_vessel_description/urdf/dlr_vessel.urdf.xacro (robot description, xacro)
@@ -1,4 +1,4 @@
 <?xml version="1.0"?>
-<robot xmlns:xacro="http://www.ros.org/wiki/xacro" name="canal_bridge">
+<robot xmlns:xacro="http://www.ros.org/wiki/xacro" name="dlr_vessel">
     <!-- Model parameters -->
     <xacro:arg name="model_name" default="model_name"/>
@@ -14,10 +14,10 @@
     </xacro:macro>
     <!-- URDF object macro -->
-    <xacro:macro name="canal_bridge" params="model_prefix">
+    <xacro:macro name="dlr_vessel" params="model_prefix">
         <material name="White">
             <color rgba="0.6 0.6 0.6 1.0"/>
         </material>
         <link name="world"/>
-        <link name="${model_prefix}main_link">
+        <link name="${model_prefix}base_link">
             <!-- <xacro:box_inertial x="0.05" y="0.05" z="0.05" mass="3.0">
                 <origin xyz="0 0 0.05" rpy="0 0 0" />
@@ -26,7 +26,7 @@
                 <origin xyz="0 0 0" rpy="0 0 0"/>
                 <geometry>
-                    <mesh filename="package://dlr_gazebo_world/meshes/canal_bridge.stl" scale="100 100 100"/>
-                    <!-- <mesh filename="package://dlr_gazebo_world/meshes/canal_bridge1.stl" scale="1000 1000 1000"/> -->
-                    <!-- <mesh filename="package://dlr_gazebo_world/meshes/canal_bridge1.stl" scale="0.001 0.001 0.001"/> -->
+                    <!-- <mesh filename="package://dlr_vessel_description/meshes/patrol_boat.stl" scale="1 1 1"/> -->
+                    <mesh filename="package://dlr_vessel_description/meshes/dlr_vessel.stl" scale="100 100 100"/>
+                    <!-- <mesh filename="package://dlr_vessel_description/meshes/dlr_vessel.stl" scale="0.001 0.001 0.001"/> -->
                 </geometry>
                 <material name="White"/>
@@ -35,5 +35,5 @@
                 <origin xyz="0 0 0.05" rpy="0 0 0"/>
                 <geometry>
-                    <mesh filename="package://dlr_gazebo_world/meshes/canal_bridge.stl" scale="100 100 100"/>
+                    <mesh filename="package://dlr_vessel_description/meshes/patrol_boat.stl" scale="100 100 100"/>
                 </geometry>
             </collision>
@@ -41,8 +41,8 @@
         <joint name="${model_prefix}base_joint" type="fixed">
             <parent link="world"/>
-            <child link="${model_prefix}main_link"/>
+            <child link="${model_prefix}base_link"/>
         </joint>
         <!-- Gazebo properties -->
-        <gazebo reference="${model_prefix}main_link">
+        <gazebo reference="${model_prefix}base_link">
             <material>Gazebo/Red</material>
             <mu1>0.2</mu1>
@@ -57,4 +57,4 @@
     </xacro:macro>
     <!-- Create macro -->
-    <xacro:canal_bridge model_prefix="$(arg model_name)_"/>
+    <xacro:dlr_vessel model_prefix="$(arg model_name)_"/>
 </robot>

Commit message: Minor changes

File: dlr_vessel_description/urdf/dlr_vessel.urdf.xacro (robot description, xacro)
@@ -20,7 +20,7 @@
         <link name="${model_prefix}base_footprint"/>
         <link name="${model_prefix}base_link">
-            <!-- <xacro:box_inertial x="0.05" y="0.05" z="0.05" mass="3.0">
-                <origin xyz="0 0 0.05" rpy="0 0 0" />
-            </xacro:box_inertial> -->
+            <xacro:box_inertial x="10" y="3" z="3" mass="1000">
+                <origin xyz="0 0 0" rpy="0 0 0" />
+            </xacro:box_inertial>
             <visual>
                 <origin xyz="0 0 0" rpy="0 0 0"/>
@@ -58,4 +58,5 @@
             <odometryRate>20.0</odometryRate>
             <robotBaseFrame>${model_prefix}base_footprint</robotBaseFrame>
+            <robotBaseFrame>${model_prefix}base_footprint</robotBaseFrame>
             </plugin>
         </gazebo>

Commit message: Modified spawn world and vessel launch files

File: dlr_vessel_description/urdf/dlr_vessel.urdf.xacro (robot description, xacro)
@@ -38,4 +38,5 @@
         </link>
         <joint name="${model_prefix}base_link_joint" type="fixed">
+            <origin xyz="0 0 0" rpy="0 0 0"/>
             <parent link="${model_prefix}base_footprint"/>
             <child link="${model_prefix}base_link"/>
@@ -50,5 +51,5 @@
             <!-- <static>true</static>   -->
         </gazebo>
-        <!-- Added the planar move plugin -->
+        <!-- Planar move plugin -->
         <gazebo>
             <plugin name="${model_prefix}planar_move_controller" filename="libdlr_gazebo_ros_planar_move.so">
