Commit message: Fixed dlr_cartographer 2D

File: dlr_vessel_description/robots/dlr_vessel.xacro (robot description, xacro)
@@ -12,5 +12,5 @@
         organize_cloud="false" hz="10" lasers="16" samples="1875"
         collision_range="0.3" min_range="0.9" max_range="130.0"
-        noise="0.008" min_angle="-${M_PI}" max_angle="${M_PI}" gpu="true">
+        noise="0.008" min_angle="-${M_PI/2}" max_angle="${M_PI/2}" gpu="true">
         <origin xyz="9.75 0 2.20" rpy="0 0 0"/>
     </xacro:VLP-16>
@@ -27,5 +27,6 @@
     <xacro:include filename="$(find dlr_sensors)/urdf/GNSS_MTi_680G.urdf.xacro" />
     <xacro:gnss_mti_680g prefix="$(arg imu_name)" parent="$(arg model_name)_base_link">
-        <origin xyz="9.75 0 2.4" rpy="0 0 0"/>
+        <!-- <origin xyz="9.75 0 2.4" rpy="0 0 0"/> -->
+        <origin xyz="0 0 0" rpy="0 0 0"/>
     </xacro:gnss_mti_680g>
 </robot>
