Commit message: Muinor changes

File: dlr_gazebo_world/urdf/canal_bridge.urdf.xacro (robot description, xacro)
@@ -15,5 +15,8 @@
     <!-- URDF object macro -->
     <xacro:macro name="canal_bridge" params="model_prefix">
-        <link name="${model_prefix}base_link"/>
+        <material name="White">
+            <color rgba="0.6 0.6 0.6 1.0"/>
+        </material>
+        <link name="world"/>
         <link name="${model_prefix}main_link">
             <!-- <xacro:box_inertial x="0.05" y="0.05" z="0.05" mass="3.0">
@@ -23,18 +26,19 @@
                 <origin xyz="0 0 0" rpy="0 0 0"/>
                 <geometry>
-                    <mesh filename="package://dlr_gazebo_world/meshes/canal_bridge1.stl" scale="1 1 1"/>
+                    <mesh filename="package://dlr_gazebo_world/meshes/canal_bridge.stl" scale="100 100 100"/>
                     <!-- <mesh filename="package://dlr_gazebo_world/meshes/canal_bridge1.stl" scale="1000 1000 1000"/> -->
                     <!-- <mesh filename="package://dlr_gazebo_world/meshes/canal_bridge1.stl" scale="0.001 0.001 0.001"/> -->
                 </geometry>
+                <material name="White"/>
             </visual>
             <collision>
                 <origin xyz="0 0 0.05" rpy="0 0 0"/>
                 <geometry>
-                    <mesh filename="package://dlr_gazebo_world/meshes/canal_bridge1.stl" scale="0.1 0.1 0.1"/>
+                    <mesh filename="package://dlr_gazebo_world/meshes/canal_bridge.stl" scale="100 100 100"/>
                 </geometry>
             </collision>
         </link>
         <joint name="${model_prefix}base_joint" type="fixed">
-            <parent link="${model_prefix}base_link"/>
+            <parent link="world"/>
             <child link="${model_prefix}main_link"/>
         </joint>

Commit message: Minor changes to dlr vessel

File: dlr_gazebo_world/urdf/canal_bridge.urdf.xacro (robot description, xacro)
@@ -27,6 +27,4 @@
                 <geometry>
                     <mesh filename="package://dlr_gazebo_world/meshes/canal_bridge.stl" scale="100 100 100"/>
-                    <!-- <mesh filename="package://dlr_gazebo_world/meshes/canal_bridge1.stl" scale="1000 1000 1000"/> -->
-                    <!-- <mesh filename="package://dlr_gazebo_world/meshes/canal_bridge1.stl" scale="0.001 0.001 0.001"/> -->
                 </geometry>
                 <material name="White"/>

File: dlr_vessel_description/urdf/dlr_vessel.urdf.xacro (robot description, xacro)
@@ -18,5 +18,5 @@
             <color rgba="0.6 0.6 0.6 1.0"/>
         </material>
-        <link name="world"/>
+        <link name="${model_prefix}base_footprint"/>
         <link name="${model_prefix}base_link">
             <!-- <xacro:box_inertial x="0.05" y="0.05" z="0.05" mass="3.0">
@@ -26,7 +26,5 @@
                 <origin xyz="0 0 0" rpy="0 0 0"/>
                 <geometry>
-                    <!-- <mesh filename="package://dlr_vessel_description/meshes/patrol_boat.stl" scale="1 1 1"/> -->
-                    <mesh filename="package://dlr_vessel_description/meshes/dlr_vessel.stl" scale="100 100 100"/>
-                    <!-- <mesh filename="package://dlr_vessel_description/meshes/dlr_vessel.stl" scale="0.001 0.001 0.001"/> -->
+                    <mesh filename="package://dlr_vessel_description/meshes/patrol_boat.stl"/>
                 </geometry>
                 <material name="White"/>
@@ -35,10 +33,10 @@
                 <origin xyz="0 0 0.05" rpy="0 0 0"/>
                 <geometry>
-                    <mesh filename="package://dlr_vessel_description/meshes/patrol_boat.stl" scale="100 100 100"/>
+                    <mesh filename="package://dlr_vessel_description/meshes/patrol_boat.stl"/>
                 </geometry>
             </collision>
         </link>
-        <joint name="${model_prefix}base_joint" type="fixed">
-            <parent link="world"/>
+        <joint name="${model_prefix}base_link_joint" type="fixed">
+            <parent link="${model_prefix}base_footprint"/>
             <child link="${model_prefix}base_link"/>
         </joint>
@@ -52,9 +50,16 @@
             <static>true</static>
         </gazebo>
+        <!-- Adde the planar move plugin -->
         <gazebo>
-            <static>true</static>
+            <plugin name="object_controller" filename="libgazebo_ros_planar_move.so">
+            <commandTopic>cmd_vel</commandTopic>
+            <odometryTopic>odom</odometryTopic>
+            <odometryFrame>odom</odometryFrame>
+            <odometryRate>20.0</odometryRate>
+            <robotBaseFrame>${model_prefix}base_footprint</robotBaseFrame>
+            </plugin>
         </gazebo>
     </xacro:macro>
     <!-- Create macro -->
-    <xacro:dlr_vessel model_prefix="$(arg model_name)_"/>
+    <!-- <xacro:dlr_vessel model_prefix="$(arg model_name)_"/> -->
 </robot>

Commit message: Added canal bridge v2 | Tested planar move gazebo plugin

File: dlr_gazebo_world/urdf/canal_bridge.urdf.xacro (robot description, xacro)
@@ -2,5 +2,5 @@
 <robot xmlns:xacro="http://www.ros.org/wiki/xacro" name="canal_bridge">
     <!-- Model parameters -->
-    <xacro:arg name="model_name" default="model_name"/>
+    <xacro:arg name="model_name" default="canal_bridge"/>
     <!-- Box inertial macro -->
     <xacro:macro name="box_inertial" params="x y z mass *origin">
@@ -18,30 +18,30 @@
             <color rgba="0.6 0.6 0.6 1.0"/>
         </material>
-        <link name="world"/>
-        <link name="${model_prefix}main_link">
-            <!-- <xacro:box_inertial x="0.05" y="0.05" z="0.05" mass="3.0">
-                <origin xyz="0 0 0.05" rpy="0 0 0" />
-            </xacro:box_inertial> -->
+        <link name="${model_prefix}base_footprint"/>
+        <link name="${model_prefix}base_link">
+            <xacro:box_inertial x="10" y="3" z="3" mass="1000">
+                <origin xyz="0 0 0" rpy="0 0 0" />
+            </xacro:box_inertial>
             <visual>
                 <origin xyz="0 0 0" rpy="0 0 0"/>
                 <geometry>
-                    <mesh filename="package://dlr_gazebo_world/meshes/canal_bridge.stl" scale="100 100 100"/>
+                    <mesh filename="package://dlr_gazebo_world/meshes/canal_bridge_2.stl" scale="200 200 200"/>
                 </geometry>
                 <material name="White"/>
             </visual>
             <collision>
-                <origin xyz="0 0 0.05" rpy="0 0 0"/>
+                <origin xyz="0 0 0" rpy="0 0 0"/>
                 <geometry>
-                    <mesh filename="package://dlr_gazebo_world/meshes/canal_bridge.stl" scale="100 100 100"/>
+                    <mesh filename="package://dlr_gazebo_world/meshes/canal_bridge_2.stl" scale="1 1 1 "/>
                 </geometry>
             </collision>
         </link>
-        <joint name="${model_prefix}base_joint" type="fixed">
-            <parent link="world"/>
-            <child link="${model_prefix}main_link"/>
+        <joint name="${model_prefix}base_link_joint" type="fixed">
+            <parent link="${model_prefix}base_footprint"/>
+            <child link="${model_prefix}base_link"/>
         </joint>
         <!-- Gazebo properties -->
-        <gazebo reference="${model_prefix}main_link">
-            <material>Gazebo/Red</material>
+        <gazebo reference="${model_prefix}base_link">
+            <material>Gazebo/Grey</material>
             <mu1>0.2</mu1>
             <mu2>0.2</mu2>
@@ -50,7 +50,4 @@
             <static>true</static>
         </gazebo>
-        <gazebo>
-            <static>true</static>
-        </gazebo>
     </xacro:macro>
     <!-- Create macro -->

File: dlr_vessel_description/robots/dlr_vessel.xacro (robot description, xacro)
@@ -12,5 +12,5 @@
         organize_cloud="false" hz="10" lasers="16" samples="1875"
         collision_range="0.3" min_range="0.9" max_range="130.0"
-        noise="0.008" min_angle="-${M_PI}" max_angle="${M_PI}" gpu="false">
+        noise="0.008" min_angle="-${M_PI}" max_angle="${M_PI}" gpu="true">
         <origin xyz="9.75 0 2.20" rpy="0 0 0"/>
     </xacro:VLP-16>

File: dlr_vessel_description/urdf/dlr_vessel.urdf.xacro (robot description, xacro)
@@ -50,7 +50,7 @@
             <!-- <static>true</static>   -->
         </gazebo>
-        <!-- Adde the planar move plugin -->
+        <!-- Added the planar move plugin -->
         <gazebo>
-            <plugin name="${model_prefix}planar_move_controller" filename="libgazebo_ros_planar_move.so">
+            <plugin name="${model_prefix}planar_move_controller" filename="libdlr_gazebo_ros_planar_move.so">
             <commandTopic>cmd_vel</commandTopic>
             <odometryTopic>odom</odometryTopic>

Commit message: Modified canal bridge gazebo world

File: dlr_gazebo_world/urdf/canal_bridge.urdf.xacro (robot description, xacro)
@@ -26,5 +26,5 @@
                 <origin xyz="0 0 0" rpy="0 0 0"/>
                 <geometry>
-                    <mesh filename="package://dlr_gazebo_world/meshes/canal_bridge_2.stl" scale="200 200 200"/>
+                    <mesh filename="package://dlr_gazebo_world/meshes/canal_bridge_2.stl" scale="250 250 250"/>
                 </geometry>
                 <material name="White"/>
@@ -33,5 +33,5 @@
                 <origin xyz="0 0 0" rpy="0 0 0"/>
                 <geometry>
-                    <mesh filename="package://dlr_gazebo_world/meshes/canal_bridge_2.stl" scale="1 1 1 "/>
+                    <mesh filename="package://dlr_gazebo_world/meshes/canal_bridge_2.stl" scale="250 250 250"/>
                 </geometry>
             </collision>
